Commit message: Added matlab position support and initial commit

File: rotors_description/urdf/ardrone.xacro (robot description, xacro)
@@ -21,4 +21,5 @@
   <xacro:property name="cos30" value="0.866025403784" />
   <xacro:property name="sqrt2" value="1.4142135623730951" />
+  <!-- <xacro:property name="sqrt2" value="0.70710678118" /> -->
   <xacro:property name="rotor_drag_coefficient" value="8.06428e-05" />
   <xacro:property name="rolling_moment_coefficient" value="0.000001" />
